File: simpleJtag/simpleJtag.sch (KiCad schematic (older format))
At the start: 11 parts

Commit message: end of day sync
Parts:
- removed U?: CH552G, symbol MCU_WCH:CH552G
- added C?: 0.1uf, symbol Device:C_Small
- added C?: 0.1uF, symbol Device:C_Small
- added D?: LED, symbol Device:LED
- added R? (x2): R_Small, symbol Device:R_Small
- added U?: CH552T, symbol MCU_WCH:CH552T
Connections:
- net labels added: RESET, TCK, TDI, TDO, TMS
- wire segments 44 -> 65
Other:
- note added: "P1.0 - TMS\n\nP1.4 & P1.7 - TCK\n\nP1.5 - TDI\n\nP1.6 - TDO"

Commit message: more schmatics work routing almost complete
Parts:
- removed R?: R_Small, symbol Device:R_Small
- added C5, C7: 1uF, Capacitor_SMD:C_0603_1608Metric, symbol Device:C_Small
- added R1: 56K, Resistor_SMD:R_0603_1608Metric, symbol Device:R_Small
- added R4: R_Small, Resistor_SMD:R_0603_1608Metric, symbol Device:R_Small
- added TP1: RESET, TestPoint:TestPoint_Pad_D2.5mm, symbol Connector:TestPoint
- added TP2: P3.3, TestPoint:TestPoint_Pad_D2.5mm, symbol Connector:TestPoint
- added TP3: P3.4, TestPoint:TestPoint_Pad_D2.5mm, symbol Connector:TestPoint
- added TP4: P3.5, TestPoint:TestPoint_Pad_D2.5mm, symbol Connector:TestPoint
- added TP5: P1.2, TestPoint:TestPoint_Pad_D2.5mm, symbol Connector:TestPoint
- added TP6: P1.3, TestPoint:TestPoint_Pad_D2.5mm, symbol Connector:TestPoint
- added TP7: P3.1, TestPoint:TestPoint_Pad_D2.5mm, symbol Connector:TestPoint
- added TP8: P3.0, TestPoint:TestPoint_Pad_D2.5mm, symbol Connector:TestPoint
- added TP9: P3.2, TestPoint:TestPoint_Pad_D2.5mm, symbol Connector:TestPoint
- C1, C2: renamed from C?; value C_Small -> 1uF; footprint (none) -> Capacitor_SMD:C_0603_1608Metric
- C3, C4: renamed from C?; footprint (none) -> Capacitor_SMD:C_0603_1608Metric
- C6: renamed from C?; value C_Small -> 0.1uF; footprint (none) -> Capacitor_SMD:C_0603_1608Metric
- D1, D2: renamed from D?; footprint (none) -> LED_SMD:LED_0805_2012Metric
- F1: renamed from F?; footprint (none) -> Capacitor_SMD:C_1210_3225Metric
- J1: renamed from J?; footprint (none) -> Connectors_Multicomp:Multicomp_MC9A22-1034_2x05x2.54mm_Angled
- JP1: renamed from JP?; footprint (none) -> Connector_PinHeader_2.54mm:PinHeader_1x03_P2.54mm_Vertical
- P1: renamed from P?; footprint (none) -> Connector_USB:USB_C_Plug_Molex_105444
- R2, R3: renamed from R?; value R_Small -> 330R; footprint (none) -> Resistor_SMD:R_0603_1608Metric
- U2: renamed from U?; footprint (none) -> Housings_SSOP:TSSOP-20_4.4x6.5mm_Pitch0.65mm
- gave numbers to parts that had none: 1
Connections:
- net labels added: J_RESET, TVCC
- wire segments 65 -> 114

Commit message: swapping USBC plug to USBC socket
Parts:
- P1: footprint Connector_USB:USB_C_Plug_Molex_105444 -> Connector_USB:USB_C_Receptacle_Amphenol_12401610E4-2A_CircularHoles
Changed lines of the file:
@@
 F 0 "P1" H 1405 3767 50  0000 C CNN
 F 1 "USB_C_Plug" H 1405 3676 50  0000 C CNN
-F 2 "Connector_USB:USB_C_Plug_Molex_105444" H 1450 2200 50  0001 C CNN
+F 2 "Connector_USB:USB_C_Receptacle_Amphenol_12401610E4-2A_CircularHoles" H 1450 2200 50  0001 C CNN
 F 3 "http://www.usb.org/developers/docs/usb_31_033017.zip" H 1450 2200 50  0001 C CNN
 	1    1300 2200

Commit message: end of day sync
Parts:
- P1: footprint Connector_USB:USB_C_Receptacle_Amphenol_12401610E4-2A_CircularHoles -> footprint:usbc_16pos_lugged_allsmt
Changed lines of the file:
@@
 F 0 "P1" H 1405 3767 50  0000 C CNN
 F 1 "USB_C_Plug" H 1405 3676 50  0000 C CNN
-F 2 "Connector_USB:USB_C_Receptacle_Amphenol_12401610E4-2A_CircularHoles" H 1450 2200 50  0001 C CNN
+F 2 "footprint:usbc_16pos_lugged_allsmt" H 1450 2200 50  0001 C CNN
 F 3 "http://www.usb.org/developers/docs/usb_31_033017.zip" H 1450 2200 50  0001 C CNN
 	1    1300 2200

Commit message: end of day sync
Parts:
- removed TP2: P3.3, TestPoint:TestPoint_Pad_D2.5mm, symbol Connector:TestPoint
- removed TP3: P3.4, TestPoint:TestPoint_Pad_D2.5mm, symbol Connector:TestPoint
- removed TP4: P3.5, TestPoint:TestPoint_Pad_D2.5mm, symbol Connector:TestPoint
- removed TP5: P1.2, TestPoint:TestPoint_Pad_D2.5mm, symbol Connector:TestPoint
- removed TP6: P1.3, TestPoint:TestPoint_Pad_D2.5mm, symbol Connector:TestPoint
- removed TP7: P3.1, TestPoint:TestPoint_Pad_D2.5mm, symbol Connector:TestPoint
- removed TP8: P3.0, TestPoint:TestPoint_Pad_D2.5mm, symbol Connector:TestPoint
- removed TP9: P3.2, TestPoint:TestPoint_Pad_D2.5mm, symbol Connector:TestPoint
- added C8, C9: 22pf, Capacitor_SMD:C_0603_1608Metric, symbol Device:C_Small
- added Y1: Crystal_GND24, symbol Device:Crystal_GND24
Connections:
- wire segments 114 -> 131
Changed lines of the file:
@@
 $EndComp
-Wire Wire Line
-	7950 4650 7200 4650
-Wire Wire Line
-	6850 4500 7400 4500
 Wire Wire Line
 	7950 4500 8350 4500
@@
 	0    1    1    0
 $EndComp
-Wire Wire Line
-	6850 4800 7600 4800
 $Comp
 L power:VBUS #PWR0111
@@
 	6850 5250 7200 5250
 Wire Wire Line
-	6850 3300 7300 3300
-Wire Wire Line
-	6850 3450 7300 3450
-$Comp
-L Connector:TestPoint TP2
-U 1 1 5E553F09
-P 7200 4950
-F 0 "TP2" V 7154 5138 50  0000 L CNN
-F 1 "P3.3" V 7245 5138 50  0000 L CNN
-F 2 "TestPoint:TestPoint_Pad_D2.5mm" H 7400 4950 50  0001 C CNN
-F 3 "~" H 7400 4950 50  0001 C CNN
-	1    7200 4950
-	0    1    1    0
-$EndComp
-$Comp
-L Connector:TestPoint TP3
-U 1 1 5E55F92F
-P 7200 5100
-F 0 "TP3" V 7154 5288 50  0000 L CNN
-F 1 "P3.4" V 7245 5288 50  0000 L CNN
-F 2 "TestPoint:TestPoint_Pad_D2.5mm" H 7400 5100 50  0001 C CNN
-F 3 "~" H 7400 5100 50  0001 C CNN
-	1    7200 5100
-	0    1    1    0
-$EndComp
-$Comp
-L Connector:TestPoint TP4
-U 1 1 5E55F96F
-P 7200 5250
-F 0 "TP4" V 7154 5438 50  0000 L CNN
-F 1 "P3.5" V 7245 5438 50  0000 L CNN
-F 2 "TestPoint:TestPoint_Pad_D2.5mm" H 7400 5250 50  0001 C CNN
-F 3 "~" H 7400 5250 50  0001 C CNN
-	1    7200 5250
-	0    1    1    0
-$EndComp
-$Comp
-L Connector:TestPoint TP5
-U 1 1 5E55F9AF
-P 7300 3300
-F 0 "TP5" V 7254 3488 50  0000 L CNN
-F 1 "P1.2" V 7345 3488 50  0000 L CNN
-F 2 "TestPoint:TestPoint_Pad_D2.5mm" H 7500 3300 50  0001 C CNN
-F 3 "~" H 7500 3300 50  0001 C CNN
-	1    7300 3300
-	0    1    1    0
-$EndComp
-$Comp
-L Connector:TestPoint TP6
-U 1 1 5E55FA2D
-P 7300 3450
-F 0 "TP6" V 7254 3638 50  0000 L CNN
-F 1 "P1.3" V 7345 3638 50  0000 L CNN
-F 2 "TestPoint:TestPoint_Pad_D2.5mm" H 7500 3450 50  0001 C CNN
-F 3 "~" H 7500 3450 50  0001 C CNN
-	1    7300 3450
-	0    1    1    0
-$EndComp
-$Comp
-L Connector:TestPoint TP8
-U 1 1 5E55FDC0
-P 7400 4500
-F 0 "TP8" H 7458 4620 50  0000 L CNN
-F 1 "P3.0" H 7458 4529 50  0000 L CNN
-F 2 "TestPoint:TestPoint_Pad_D2.5mm" H 7600 4500 50  0001 C CNN
-F 3 "~" H 7600 4500 50  0001 C CNN
-	1    7400 4500
-	1    0    0    -1
-$EndComp
-Connection ~ 7400 4500
-Wire Wire Line
-	7400 4500 7650 4500
-$Comp
-L Connector:TestPoint TP7
-U 1 1 5E55FF37
-P 7200 4650
-F 0 "TP7" H 7258 4770 50  0000 L CNN
-F 1 "P3.1" H 7258 4679 50  0000 L CNN
-F 2 "TestPoint:TestPoint_Pad_D2.5mm" H 7400 4650 50  0001 C CNN
-F 3 "~" H 7400 4650 50  0001 C CNN
-	1    7200 4650
-	1    0    0    -1
-$EndComp
-Connection ~ 7200 4650
-Wire Wire Line
-	7200 4650 6850 4650
-$Comp
-L Connector:TestPoint TP9
-U 1 1 5E55FFD5
-P 7600 4800
-F 0 "TP9" H 7542 4827 50  0000 R CNN
-F 1 "P3.2" H 7542 4918 50  0000 R CNN
-F 2 "TestPoint:TestPoint_Pad_D2.5mm" H 7800 4800 50  0001 C CNN
-F 3 "~" H 7800 4800 50  0001 C CNN
-	1    7600 4800
-	-1   0    0    1
-$EndComp
-Connection ~ 7600 4800
-Wire Wire Line
-	7600 4800 7650 4800
+	6850 3300 7250 3300
+Wire Wire Line
+	6850 3450 7250 3450
+Wire Wire Line
+	7250 3300 7250 3200
+Wire Wire Line
+	7250 3450 7250 3500
+Wire Wire Line
+	8150 3500 8150 3350
+Wire Wire Line
+	8050 3200 8050 3050
+Wire Wire Line
+	8050 3050 8550 3050
+Wire Wire Line
+	8550 3050 8550 3350
+Wire Wire Line
+	8550 3350 8450 3350
+Wire Wire Line
+	7250 3200 8050 3200
+Wire Wire Line
+	7250 3500 8050 3500
+$Comp
+L Device:C_Small C9
+U 1 1 5E58319E
+P 8550 3600
+F 0 "C9" H 8642 3646 50  0000 L CNN
+F 1 "22pf" H 8642 3555 50  0000 L CNN
+F 2 "Capacitor_SMD:C_0603_1608Metric" H 8550 3600 50  0001 C CNN
+F 3 "~" H 8550 3600 50  0001 C CNN
+	1    8550 3600
+	1    0    0    -1
+$EndComp
+$Comp
+L Device:C_Small C8
+U 1 1 5E5832C0
+P 8050 3600
+F 0 "C8" H 8142 3646 50  0000 L CNN
+F 1 "22pf" H 8142 3555 50  0000 L CNN
+F 2 "Capacitor_SMD:C_0603_1608Metric" H 8050 3600 50  0001 C CNN
+F 3 "~" H 8050 3600 50  0001 C CNN
+	1    8050 3600
+	1    0    0    -1
+$EndComp
+Connection ~ 8050 3500
+Wire Wire Line
+	8050 3500 8150 3500
+Wire Wire Line
+	8050 3700 8050 3850
+Wire Wire Line
+	8050 3850 8300 3850
+Wire Wire Line
+	8550 3850 8550 3700
+Wire Wire Line
+	8300 3550 8300 3850
+Connection ~ 8300 3850
+Wire Wire Line
+	8300 3850 8500 3850
+Wire Wire Line
+	8300 3150 8300 3100
+Wire Wire Line
+	8300 3100 8500 3100
+Wire Wire Line
+	8500 3100 8500 3850
+Connection ~ 8500 3850
+Wire Wire Line
+	8500 3850 8550 3850
+Wire Wire Line
+	8550 3350 8550 3500
+Connection ~ 8550 3350
+$Comp
+L power:GND #PWR0120
+U 1 1 5E592E6E
+P 8300 3850
+F 0 "#PWR0120" H 8300 3600 50  0001 C CNN
+F 1 "GND" H 8305 3677 50  0000 C CNN
+F 2 "" H 8300 3850 50  0001 C CNN
+F 3 "" H 8300 3850 50  0001 C CNN
+	1    8300 3850
+	1    0    0    -1
+$EndComp
+Wire Wire Line
+	6850 4500 7650 4500
+Wire Wire Line
+	6850 4650 7950 4650
+Wire Wire Line
+	6850 4800 7650 4800
+$Comp
+L Device:Crystal_GND24 Y1
+U 1 1 5E593996
+P 8300 3350
+F 0 "Y1" H 8491 3396 50  0000 L CNN
+F 1 "Crystal_GND24" H 8491 3305 50  0000 L CNN
+F 2 "" H 8300 3350 50  0001 C CNN
+F 3 "~" H 8300 3350 50  0001 C CNN
+	1    8300 3350
+	1    0    0    -1
+$EndComp
 $EndSCHEMATC
